File: hardware/time-twister.brd (EAGLE design)
At the start: 154.9 x 82.5 mm, 86 parts, among them IC1 MEGA8-AI, IC2 7805T, IC3 6N138, IC4 74HC14D, X1 HD44780LCD-1602

Commit message: updates
Parts:
- removed C200, C201, C202, C203, C204, C205: (no value), rcl:C0805
- removed D107: 0805DIODE, jasons_stuff:0805DIODE
- removed Q1: (no value), crystal:HC49/S
- removed R202, R203, R204, R205: (no value), rcl:M0805
- added C10, C11: (no value), rcl:E2,5-6
- added C12, C13, C40, C9: (no value), rcl:C0805
- added D9: 0805DIODE, jasons_stuff:0805DIODE
- added LCD: HD44780LCD-1602, adafruit:LCD1602
- added R10, R11, R18, R7: (no value), rcl:R0805
- C7, C8: device rcl:E2,5-6 -> rcl:C0805
- R2, R3, R4, R5: device rcl:R0805 -> rcl:M0805
- X1: value HD44780LCD-1602 -> (none); device adafruit:LCD1602 -> crystal:HC49/S
- moved R1 103.3 mm to (133.9, 80.0)
- moved R12 103.3 mm to (36.8, 44.5)
- moved D5 94.0 mm to (113.0, 31.8), turned to 0 degrees
- moved C8 90.9 mm to (63.5, 62.2), turned to 90 degrees
- moved C1 75.5 mm to (99.1, 87.6), turned to 180 degrees
- moved R5 73.7 mm to (68.6, 87.6), turned to 0 degrees
- moved C7 69.5 mm to (85.6, 53.6)
- moved C6 64.6 mm to (94.0, 73.0), turned to 0 degrees
- moved R4 52.8 mm to (81.3, 87.6), turned to 0 degrees
- moved C4 51.7 mm to (61.0, 87.6), turned to 180 degrees
- moved C5 50.5 mm to (48.3, 87.6), turned to 180 degrees
- moved C2 34.2 mm to (86.4, 87.6), turned to 180 degrees
- moved C3 33.3 mm to (73.7, 87.6), turned to 180 degrees
- moved X1 33.3 mm to (67.6, 59.2), flipped to the bottom, turned to 270 degrees
- moved R8 22.7 mm to (91.4, 77.2), turned to 180 degrees
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- renumbered BEAT to SYNC, CLK_OUT_A to OUT_A, CLK_OUT_B to OUT_B, CLK_OUT_C to OUT_C, CLK_OUT_D to OUT_D, D100 to D12, D101 to D10, D102 to D13, D103 to D11, D104 to D8, D105 to D7, D106 to D6, LED1 to PWR, R201 to R6, R21 to R9, R700 to R16, R701 to R17, R702 to R14, R703 to R13, R704 to R15, SERIAL_PROG to SERIAL, T1 to TR1, U$1 to ENC1, U$3 to ONOFF
Connections:
- net DB4: now also LCD.11; no longer X1.11
- net DB5: now also LCD.12; no longer X1.12
- net DB6: now also LCD.13; no longer X1.13
- net DB7: now also LCD.14; no longer X1.14
- net E: now also LCD.6; no longer X1.6
- net GND: now also C1.1, C10.-, C11.-, C12.1, C13.2, C4.1, C7.1, C8.1, C9.1, D1.A, LCD.1, LCD.16, LCD.5, R1.2, R10.2, R11.2, R18.2; no longer C1.2, C200.1, C201.1, C202.1, C203.1, C204.1, C205.1, C7.-, C8.-, D2.A, R12.2, R4.2, R5.2, R8.2, X1.1, X1.16, X1.5
- net INDC: now also R7.2; no longer R2.2
- net KEY_RET1: now also R11.1; no longer R4.1
- net KEY_RET2: now also D5.A, R18.1; no longer D107.A, R5.1
- net LCD_A: now also LCD.15, R8.1; no longer R3.1, X1.15
- net LCD_VO: now also LCD.3; no longer X1.3
- net MIDI_OUT_5: now also D9.C; no longer D5.C
- net N$12: now also C10.+, C12.2, D2.C; no longer C6.2, C8.+, D1.C
- net N$13: now also C4.2, R5.2; no longer C202.2, R202.2
- net N$14: now also C2.2, R3.2; no longer C204.2, R204.2
- net N$15: now also C1.2, R2.2; no longer C205.2, R205.2
- net N$17: now also C5.2; no longer C201.2
- net N$21: now also R7.1; no longer R2.1
- net N$24: now also R2.1; no longer R205.1
- net N$25: now also R3.1; no longer R204.1
- net N$26: now also R4.1; no longer R203.1
- net N$27: now also R5.1; no longer R202.1
- net N$33: now also D5.C; no longer D107.C
- net N$4: now also C9.2, X1.2; no longer C3.2, Q1.2
- net N$45: now also D9.A; no longer D5.A
- net N$5: now also C8.2, X1.1; no longer C2.2, Q1.1
- net N$50: now also R10.1; no longer R8.1
- net N$51: now also R1.1; no longer R12.1
- net N$55: now also D1.C, D2.A; no longer D3.A, D4.C
- net N$56: now also D3.A, D4.C; no longer D1.A, D2.C
- net N$6: now also C3.2, R4.2; no longer C203.2, R203.2
- net N$7: now also C40.1, R12.1; no longer C4.1, R1.1
- net N$9: now also C40.2; no longer C4.2
- net RS: now also LCD.4; no longer X1.4
- net VDD: now also C11.+, C13.1, C6.2, C7.2, LCD.2, R12.2, R8.2; no longer C1.1, C200.2, C5.2, C7.+, R1.2, R3.2, X1.2
Routing:
- net N$11: track 118.2 -> 118.7 mm
Other:
- board text added: "1"
- board text added: "BATT_9V"
- board text added: "DC_IN"
- board text added: "IN4"
- board text added: "IN5"
- board text added: "MIDI"
- board text added: "ONOFF"
- board text added: "OUT4"
- board text added: "OUT5"
- board text added: "hotchk155"
- board text added: "rev 1"
- board text added: "six4pix.com/twister"
