File: hardware/time-twister.sch (EAGLE design)
At the start: 86 parts, among them IC1 MEGA8-AI, IC2 7805T, IC3 6N138, IC4 74HC14D, X1 HD44780LCD-1602

Commit message: updates
Parts:
- removed C200, C201, C202, C203, C204, C205: (no value), rcl:C-EUC0805
- removed D107: 0805DIODE, jasons_stuff:0805DIODE
- removed Q1: (no value), crystal:CRYSTALHC49S
- removed R202, R203, R204, R205: (no value), rcl:R-EU_M0805
- added C10, C11: (no value), rcl:CPOL-EUE2.5-6
- added C12, C13, C40, C9: (no value), rcl:C-EUC0805
- added D9: 0805DIODE, jasons_stuff:0805DIODE
- added LCD: HD44780LCD-1602, adafruit:HD44780LCD-1602
- added R10, R11, R18, R7: (no value), rcl:R-EU_R0805
- C7, C8: device rcl:CPOL-EUE2.5-6 -> rcl:C-EUC0805
- R2, R3, R4, R5: device rcl:R-EU_R0805 -> rcl:R-EU_M0805
- X1: value HD44780LCD-1602 -> (none); device adafruit:HD44780LCD-1602 -> crystal:CRYSTALHC49S
- renumbered BEAT to SYNC, CLK_OUT_A to OUT_A, CLK_OUT_B to OUT_B, CLK_OUT_C to OUT_C, CLK_OUT_D to OUT_D, D100 to D12, D101 to D10, D102 to D13, D103 to D11, D104 to D8, D105 to D7, D106 to D6, LED1 to PWR, R201 to R6, R21 to R9, R700 to R16, R701 to R17, R702 to R14, R703 to R13, R704 to R15, SERIAL_PROG to SERIAL, T1 to TR1, U$1 to ENC1, U$3 to ONOFF
Connections:
- net DB4: now also LCD.DB4; no longer X1.DB4
- net DB5: now also LCD.DB5; no longer X1.DB5
- net DB6: now also LCD.DB6; no longer X1.DB6
- net DB7: now also LCD.DB7; no longer X1.DB7
- net E: now also LCD.E; no longer X1.E
- net GND: now also C1.1, C10.-, C11.-, C12.1, C13.2, C4.1, C7.1, C8.1, C9.1, D1.A, LCD.K, LCD.RW, LCD.VSS, R1.2, R10.2, R11.2, R18.2; no longer C1.2, C200.1, C201.1, C202.1, C203.1, C204.1, C205.1, C7.-, C8.-, D2.A, R12.2, R4.2, R5.2, R8.2, X1.K, X1.RW, X1.VSS
- net INDC: now also R7.2; no longer R2.2
- net KEY_RET1: now also R11.1; no longer R4.1
- net KEY_RET2: now also D5.P$2, R18.1; no longer D107.P$2, R5.1
- net LCD_A: now also LCD.A, R8.1; no longer R3.1, X1.A
- net LCD_VO: now also LCD.VO; no longer X1.VO
- net MIDI_OUT_5: now also D9.P$1; no longer D5.P$1
- net N$12: now also C10.+, C12.2, D2.C; no longer C6.2, C8.+, D1.C
- net N$13: now also C4.2, R5.2; no longer C202.2, R202.2
- net N$14: now also C2.2, R3.2; no longer C204.2, R204.2
- net N$15: now also C1.2, R2.2; no longer C205.2, R205.2
- net N$17: now also C5.2; no longer C201.2
- net N$21: now also R7.1; no longer R2.1
- net N$24: now also R2.1; no longer R205.1
- net N$25: now also R3.1; no longer R204.1
- net N$26: now also R4.1; no longer R203.1
- net N$27: now also R5.1; no longer R202.1
- net N$33: now also D5.P$1; no longer D107.P$1
- net N$4: now also C9.2, X1.2; no longer C3.2, Q1.2
- net N$45: now also D9.P$2; no longer D5.P$2
- net N$5: now also C8.2, X1.1; no longer C2.2, Q1.1
- net N$50: now also R10.1; no longer R8.1
- net N$51: now also R1.1; no longer R12.1
- net N$55: now also D1.C, D2.A; no longer D3.A, D4.C
- net N$56: now also D3.A, D4.C; no longer D1.A, D2.C
- net N$6: now also C3.2, R4.2; no longer C203.2, R203.2
- net N$7: now also C40.1, R12.1; no longer C4.1, R1.1
- net N$9: now also C40.2; no longer C4.2
- net RS: now also LCD.RS; no longer X1.RS
- net VDD: now also C11.+, C13.1, C6.2, C7.2, LCD.VDD, R12.2, R8.2; no longer C1.1, C200.2, C5.2, C7.+, R1.2, R3.2, X1.VDD
